File: HARDWARE/Inverter_Connector/Inverter_Connector.kicad_sch (KiCad schematic)
At the start: 7 parts, among them J1 M300-MV30645M1, J2 1803277, J3 1803277, J4 1894820, J5 1881451, J6 1881451, J7 1881448

Commit message: Corrected a typo
Other:
- title: Inventer_Connector -> Inverter_Connector
Changed lines of the file:
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@@
 	(paper "A4")
 	(title_block
-		(title "Inventer_Connector")
+		(title "Inverter_Connector")
 		(date "08.05.2025")
 		(rev "${REVISION}")
